File: pcb/undead_split.kicad_pcb (KiCad board)
At the start: 2 copper layers, 356.8 x 105 mm, 174 parts, among them J1 USB_C_Receptacle_USB2.0, J2 USB_C_Receptacle_USB2.0, J3 USB_C_Receptacle_USB2.0, J4 USB_C_Receptacle_USB2.0, SW1 SW_Push, SW10 SW_Push, SW11 SW_Push, SW12 SW_Push, SW13 SW_Push, SW14 SW_Push, SW15 SW_Push, SW16 SW_Push, SW17 SW_Push, SW18 SW_Push, SW19 SW_Push, SW2 SW_Push, SW20 SW_Push, SW21 SW_Push, SW22 SW_Push, SW23 SW_Push, SW24 SW_Push, SW25 SW_Push, SW26 SW_Push, SW27 SW_Push, SW28 SW_Push, SW29 SW_Push, SW3 SW_Push, SW30 SW_Push, SW31 SW_Push, SW32 SW_Push, SW33 SW_Push, SW34 SW_Push, SW35 SW_Push, SW36 SW_Push, SW37 SW_Push, SW38 SW_Push, SW39 SW_Push, SW4 SW_Push, SW40 SW_Push, SW41 SW_Push, SW42 SW_Push, SW43 SW_Push, SW44 SW_Push, SW45 SW_Push, SW46 SW_Push, SW47 SW_Push, SW48 SW_Push, SW49 SW_Push, SW5 SW_Push, SW50 SW_Push, SW51 SW_Push, SW52 SW_Push, SW53 SW_Push, SW54 SW_Push, SW55 SW_Push, SW56 SW_Push, SW57 SW_Push, SW58 SW_Push, SW59 SW_Push, SW6 SW_Push, SW60 SW_Push, SW7 SW_Push, SW8 SW_Push, SW9 SW_Push, U1 ATmega32U4-A, U2 ATmega32U4-A

Commit message: Add JLCPCB part IDs
Parts:
- J1, J2, J3, J4: footprint Connector_USB:USB_C_Receptacle_GCT_USB4105-xx-A_16P_TopMnt_Horizontal -> footprints:USB_C_Receptacle_ShouHan_16P_TopMnt_Horizontal

Commit message: Add JLCPCB production requirements
Parts:
- added H10: ToolingHole, footprints:tooling_hole, F.Cu at (204.4, 100.1)
- added H11: ToolingHole, footprints:tooling_hole, F.Cu at (39.2, 193.7)
- added H12: ToolingHole, footprints:tooling_hole, F.Cu at (204.4, 193.7)
- added H13: ToolingHole, footprints:tooling_hole, F.Cu at (222.0, 100.1)
- added H14: ToolingHole, footprints:tooling_hole, F.Cu at (387.2, 100.1)
- added H15: ToolingHole, footprints:tooling_hole, F.Cu at (387.2, 193.7)
- added H9: ToolingHole, footprints:tooling_hole, F.Cu at (39.2, 100.1)
- moved JP1 13.1 mm to (39.3, 181.4)
- moved R2 2.99 mm to (39.6, 188.5)
- moved JP2 0.88 mm to (365.5, 194.5)
- moved R8 0.88 mm to (365.5, 191.5)
Routing:
- net RESET: track 12.6 -> 19.6 mm
- net RESET-R: track 12.7 -> 13.5 mm

Commit message: Fix footprint position and rotation
This change allows for easy JLCPCB production without having to perform
any manual placement or rotation steps.
Parts:
- moved J1 1.32 mm to (49.8, 99.4)
- moved J2 1.32 mm to (193.8, 99.4)
- moved J3 1.32 mm to (376.6, 99.4)
- moved J4 1.32 mm to (232.6, 99.4)
- moved JOY1 0.83 mm to (205.8, 162.8)
- moved JOY2 0.83 mm to (244.6, 162.8)
