File: pcb/undead_split.kicad_pcb (KiCad board)
At the start: 2 copper layers, 356.8 x 105 mm, 181 parts, among them J1 USB_C_Receptacle_USB2.0, J2 USB_C_Receptacle_USB2.0, J3 USB_C_Receptacle_USB2.0, J4 USB_C_Receptacle_USB2.0, SW1 SW_Push, SW10 SW_Push, SW11 SW_Push, SW12 SW_Push, SW13 SW_Push, SW14 SW_Push, SW15 SW_Push, SW16 SW_Push, SW17 SW_Push, SW18 SW_Push, SW19 SW_Push, SW2 SW_Push, SW20 SW_Push, SW21 SW_Push, SW22 SW_Push, SW23 SW_Push, SW24 SW_Push, SW25 SW_Push, SW26 SW_Push, SW27 SW_Push, SW28 SW_Push, SW29 SW_Push, SW3 SW_Push, SW30 SW_Push, SW31 SW_Push, SW32 SW_Push, SW33 SW_Push, SW34 SW_Push, SW35 SW_Push, SW36 SW_Push, SW37 SW_Push, SW38 SW_Push, SW39 SW_Push, SW4 SW_Push, SW40 SW_Push, SW41 SW_Push, SW42 SW_Push, SW43 SW_Push, SW44 SW_Push, SW45 SW_Push, SW46 SW_Push, SW47 SW_Push, SW48 SW_Push, SW49 SW_Push, SW5 SW_Push, SW50 SW_Push, SW51 SW_Push, SW52 SW_Push, SW53 SW_Push, SW54 SW_Push, SW55 SW_Push, SW56 SW_Push, SW57 SW_Push, SW58 SW_Push, SW59 SW_Push, SW6 SW_Push, SW60 SW_Push, SW7 SW_Push, SW8 SW_Push, SW9 SW_Push, U1 ATmega32U4-A, U2 ATmega32U4-A

Commit message: Fix version on silkscreen
Other:
- board text added: "Undead Split v3 https://github.com/chrisduerr/undeadsplit"
- board text removed: "Undead Split v2 https://github.com/chrisduerr/undeadsplit"
Changed lines of the file:
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@@
 		(layer "Edge.Cuts")
 	)
-	(gr_text "Undead Split v2\nhttps://github.com/chrisduerr/undeadsplit"
+	(gr_text "Undead Split v3\nhttps://github.com/chrisduerr/undeadsplit"
 		(at 304.583462 196.938198 0)
 		(layer "B.SilkS")
@@
 		)
 	)
-	(gr_text "Undead Split v2\nhttps://github.com/chrisduerr/undeadsplit"
+	(gr_text "Undead Split v3\nhttps://github.com/chrisduerr/undeadsplit"
 		(at 121.833462 196.938198 0)
 		(layer "B.SilkS")
